File: Eagle/MyMultisensors_rev1-1.brd (EAGLE design)
At the start: 49 x 25.4 mm, 89 parts, among them Q1 SI2399DS-T1-GE3, U1 TLV3691, U2 TSU102, U3 TLV3691, U4 ATMega-328, U5 SI7021, U6 OPT3001DNP, U7 AT25DF512C_MAHNT, U8 ATSHA204A, U9 RFM69_MINIMAL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

Commit message: Reverse polarity protection fixed
Drain and source was inverted on Q1 for revision 1.0 powering through
mosfet diode (0.6V) when polarity was crossed.
Connections:
- net N$24: now also Q1.3; no longer Q1.2
- net VCC: now also Q1.2; no longer Q1.3
Routing:
- net N$24: track 55.8 -> 55.0 mm
Other:
- board text added: "Multisensors r1.1 Scalz (c) 2016"
- board text removed: "Multisensors r1 Scalz (c) 2016"
Changed lines of the file:
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@@
 <board>
 <plain>
-<text x="20.193" y="5.842" size="0.8128" layer="22" rot="MR90" align="center">Multisensors r1
+<text x="20.193" y="5.842" size="0.8128" layer="22" rot="MR90" align="center">Multisensors r1.1
 Scalz (c) 2016
 </text>
@@
 <contactref element="C26" pad="2"/>
 <contactref element="C30" pad="2"/>
-<contactref element="Q1" pad="3"/>
 <contactref element="C33" pad="2"/>
 <contactref element="C32" pad="2"/>
@@
 <wire x1="37.061" y1="4.207" x2="36.576" y2="4.357" width="0.508" layer="1"/>
 <wire x1="38.608" y1="4.357" x2="36.576" y2="4.357" width="0.508" layer="1"/>
-<wire x1="43.7642" y1="5.842" x2="40.513" y2="5.842" width="0.508" layer="1"/>
-<wire x1="40.513" y1="5.842" x2="38.989" y2="4.318" width="0.508" layer="1"/>
-<wire x1="38.989" y1="4.318" x2="38.95" y2="4.318" width="0.508" layer="1"/>
-<wire x1="38.95" y1="4.318" x2="38.608" y2="4.357" width="0.508" layer="1"/>
 <wire x1="31.623" y1="4.207" x2="31.766" y2="4.207" width="0.508" layer="1"/>
 <wire x1="31.766" y1="4.207" x2="30.607" y2="3.048" width="0.508" layer="1"/>
@@
 <wire x1="46.101" y1="17.272" x2="46.609" y2="16.764" width="0.4064" layer="1"/>
 <wire x1="46.609" y1="16.764" x2="46.609" y2="9.017" width="0.4064" layer="1"/>
-<wire x1="46.609" y1="9.017" x2="44.323" y2="6.731" width="0.4064" layer="1"/>
 <contactref element="U3" pad="5"/>
 <contactref element="C20" pad="2"/>
@@
 <wire x1="41.402" y1="15.025" x2="42.926" y2="15.025" width="0.4064" layer="1"/>
 <wire x1="42.926" y1="15.025" x2="43.092" y2="14.859" width="0.4064" layer="1"/>
-<wire x1="44.323" y1="6.731" x2="44.323" y2="6.4008" width="0.4064" layer="1"/>
-<wire x1="44.323" y1="6.4008" x2="43.7642" y2="5.842" width="0.4064" layer="1"/>
+<contactref element="Q1" pad="2"/>
+<wire x1="41.5798" y1="4.9022" x2="40.0812" y2="4.9022" width="0.508" layer="1"/>
+<wire x1="40.0812" y1="4.9022" x2="39.497" y2="4.318" width="0.508" layer="1"/>
+<wire x1="39.497" y1="4.318" x2="38.647" y2="4.318" width="0.508" layer="1"/>
+<wire x1="38.647" y1="4.318" x2="38.608" y2="4.357" width="0.508" layer="1"/>
+<wire x1="46.609" y1="9.017" x2="44.45" y2="6.858" width="0.4064" layer="1"/>
+<wire x1="44.45" y1="6.858" x2="43.18" y2="6.858" width="0.4064" layer="1"/>
+<wire x1="43.18" y1="6.858" x2="42.672" y2="6.35" width="0.4064" layer="1"/>
+<wire x1="42.672" y1="6.35" x2="42.672" y2="6.223" width="0.4064" layer="1"/>
+<wire x1="42.672" y1="6.223" x2="41.91" y2="5.461" width="0.4064" layer="1"/>
+<wire x1="41.91" y1="5.461" x2="41.91" y2="5.2324" width="0.4064" layer="1"/>
+<wire x1="41.91" y1="5.2324" x2="41.5798" y2="4.9022" width="0.4064" layer="1"/>
 </signal>
 <signal name="GND">
@@
 <contactref element="C29" pad="2"/>
 <contactref element="C30" pad="1"/>
-<contactref element="Q1" pad="1"/>
 <contactref element="BAT-" pad="1"/>
 <contactref element="D3" pad="MINUS"/>
@@
 <wire x1="31.6856" y1="17.907" x2="31.5468" y2="18.0458" width="0.4064" layer="1"/>
 <wire x1="33.147" y1="18.288" x2="31.8126" y2="18.288" width="0.4064" layer="1"/>
+<contactref element="Q1" pad="1"/>
 </signal>
 <signal name="N$3">
@@
 </signal>
 <signal name="N$24">
-<contactref element="Q1" pad="2"/>
 <contactref element="BAT+" pad="P$1"/>
 <contactref element="COIN_HOLDER" pad="VBAT@1"/>
@@
 <wire x1="35.941" y1="0.762" x2="37.592" y2="0.762" width="0.4064" layer="1"/>
 <wire x1="37.592" y1="0.762" x2="37.592" y2="0.889" width="0.4064" layer="1"/>
-<wire x1="41.5798" y1="4.9022" x2="44.7802" y2="4.9022" width="0.508" layer="1"/>
-<wire x1="44.7802" y1="4.9022" x2="45.212" y2="5.334" width="0.508" layer="1"/>
-<wire x1="45.212" y1="5.334" x2="45.212" y2="6.477" width="0.508" layer="1"/>
 <wire x1="45.212" y1="6.477" x2="45.72" y2="6.985" width="0.508" layer="1"/>
-<wire x1="41.5798" y1="4.9022" x2="41.7068" y2="3.8608" width="0.508" layer="1"/>
-<wire x1="41.7068" y1="3.8608" x2="41.148" y2="3.302" width="0.508" layer="1"/>
 <wire x1="41.148" y1="3.302" x2="37.719" y2="3.302" width="0.508" layer="1"/>
 <wire x1="37.719" y1="3.302" x2="36.957" y2="2.54" width="0.508" layer="1"/>
@@
 <wire x1="36.957" y1="0.889" x2="36.510309375" y2="0.889" width="0.254" layer="1"/>
 <wire x1="36.510309375" y1="0.889" x2="36.510309375" y2="1.042275" width="0.254" layer="1"/>
+<contactref element="Q1" pad="3"/>
+<wire x1="41.148" y1="3.302" x2="42.164" y2="3.302" width="0.508" layer="1"/>
+<wire x1="42.164" y1="3.302" x2="43.561" y2="4.699" width="0.508" layer="1"/>
+<wire x1="43.561" y1="4.699" x2="43.561" y2="5.6388" width="0.508" layer="1"/>
+<wire x1="43.561" y1="5.6388" x2="43.7642" y2="5.842" width="0.508" layer="1"/>
+<wire x1="43.7642" y1="5.842" x2="44.577" y2="5.842" width="0.508" layer="1"/>
+<wire x1="44.577" y1="5.842" x2="45.212" y2="6.477" width="0.508" layer="1"/>
 <wire x1="35.941" y1="24.638" x2="35.941" y2="24.638" width="0" layer="19" extent="1-16"/>
 <wire x1="36.449" y1="0.889" x2="36.510309375" y2="0.889" width="0" layer="19" extent="1-16"/>
