File: Eagle/MyMultisensors_rev1-1.sch (EAGLE design)
At the start: 88 parts, among them Q1 SI2399DS-T1-GE3, U1 TLV3691, U2 TSU102, U3 TLV3691, U4 ATMega-328, U5 SI7021, U6 OPT3001DNP, U7 AT25DF512C_MAHNT, U8 ATSHA204A, U9 RFM69_MINIMAL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

Commit message: Reverse polarity protection fixed
Drain and source was inverted on Q1 for revision 1.0 powering through
mosfet diode (0.6V) when polarity was crossed.
Connections:
- net N$24: now also Q1.D; no longer Q1.S
- net VCC: now also Q1.S; no longer Q1.D
Changed lines of the file:
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@@
 <instance part="C30" gate="G$1" x="-119.38" y="137.16" rot="R180"/>
 <instance part="GND39" gate="1" x="-119.38" y="121.92"/>
-<instance part="Q1" gate="A" x="-165.1" y="193.04" smashed="yes" rot="MR90">
-<attribute name="NAME" x="-167.0812" y="197.0024" size="2.0828" layer="95" ratio="10" rot="SMR0"/>
+<instance part="Q1" gate="A" x="-165.1" y="193.04" smashed="yes" rot="R90">
+<attribute name="NAME" x="-163.1188" y="197.0024" size="2.0828" layer="95" ratio="10" rot="SR0"/>
 </instance>
 <instance part="BAT+" gate="G$1" x="-187.96" y="193.04" smashed="yes" rot="R180">
@@
 </segment>
 <segment>
-<pinref part="Q1" gate="A" pin="D"/>
 <pinref part="VCC5" gate="G$1" pin="VCC"/>
-<wire x1="-160.02" y1="193.04" x2="-160.02" y2="195.58" width="0.1524" layer="91"/>
 <wire x1="-160.02" y1="195.58" x2="-160.02" y2="198.12" width="0.1524" layer="91"/>
+<pinref part="Q1" gate="A" pin="S"/>
+<wire x1="-160.02" y1="195.58" x2="-160.02" y2="193.04" width="0.1524" layer="91"/>
 </segment>
 <segment>
@@
 <pinref part="GND23" gate="1" pin="GND"/>
 <wire x1="-165.1" y1="167.64" x2="-165.1" y2="170.18" width="0.1524" layer="91"/>
-<pinref part="Q1" gate="A" pin="G"/>
-<wire x1="-165.1" y1="185.42" x2="-165.1" y2="182.88" width="0.1524" layer="91"/>
 <wire x1="-177.8" y1="170.18" x2="-175.26" y2="170.18" width="0.1524" layer="91"/>
 <pinref part="BAT-" gate="G$1" pin="1"/>
@@
 <wire x1="-175.26" y1="177.8" x2="-175.26" y2="170.18" width="0.1524" layer="91"/>
 <junction x="-175.26" y="170.18"/>
+<pinref part="Q1" gate="A" pin="G"/>
+<wire x1="-165.1" y1="182.88" x2="-165.1" y2="185.42" width="0.1524" layer="91"/>
 </segment>
 </net>
@@
 <net name="N$24" class="0">
 <segment>
-<pinref part="Q1" gate="A" pin="S"/>
 <pinref part="BAT+" gate="G$1" pin="1"/>
 <wire x1="-185.42" y1="193.04" x2="-175.26" y2="193.04" width="0.1524" layer="91"/>
-<wire x1="-175.26" y1="193.04" x2="-170.18" y2="193.04" width="0.1524" layer="91"/>
 <wire x1="-175.26" y1="193.04" x2="-175.26" y2="185.42" width="0.1524" layer="91"/>
-<junction x="-175.26" y="193.04"/>
 <pinref part="COIN_HOLDER" gate="G$1" pin="+@1"/>
-</segment>
-</net>
+<pinref part="Q1" gate="A" pin="D"/>
+<wire x1="-170.18" y1="193.04" x2="-175.26" y2="193.04" width="0.1524" layer="91"/>
+</segment>
+</net>
